File: V2/JlinkBreakout.kicad_pcb (KiCad board)
At the start: 2 copper layers, 38.5 x 27 mm, 11 parts, among them J1 JLINK, J2 TC, J3 SWD, U1 SGM2019, U2 switch_0204

Commit message: finalized V2
Parts:
- C1, C2, R1, R2, R3, R4, U1: moved to B.Cu
- J3: footprint Connector_JST:JST_XH_B4B-XH-A_1x04_P2.50mm_Vertical -> Connector_JST:JST_XH_B5B-XH-A_1x05_P2.50mm_Vertical
- moved R4 32.6 mm to (72.6, 40.2)
- moved R3 30.1 mm to (72.6, 42.8)
- moved R1 25.5 mm to (76.6, 45.4), turned to 180 degrees
- moved U2 20.6 mm to (76.6, 46.5), turned to 90 degrees
- moved R2 20.1 mm to (72.6, 52.8)
- moved C1 18.2 mm to (64.2, 54.0), turned to 90 degrees
- moved U1 17.9 mm to (67.0, 54.0)
- moved C2 17.6 mm to (69.8, 54.0), turned to 90 degrees
- moved J2 5.91 mm to (69.1, 46.3)
- moved J3 1.25 mm to (92.1, 51.5)
Connections:
- J3 pad 1: GND -> REF
- J3 pad 2: DIO -> RST
- J3 pad 3: REF -> CLK
- J3 pad 4: CLK -> DIO
Routing:
- net REF: track 0.00 -> 45.0 mm
- net RST: track 0.00 -> 39.3 mm, vias 0 -> 1
- net CLK: track 0.00 -> 39.2 mm, vias 0 -> 1
- net DIO: track 0.00 -> 34.3 mm, vias 0 -> 1
- net LDOOUT: track 0.00 -> 26.7 mm
- net +5V: track 0.00 -> 12.9 mm, vias 0 -> 1
- net SWO: track 0.00 -> 12.2 mm, vias 0 -> 1
- net Net-(R1-Pad2): track 0.00 -> 12.0 mm
- net Net-(R2-Pad2): track 0.00 -> 4.50 mm
- net Net-(R3-Pad2): track 0.00 -> 1.99 mm
- net Net-(R4-Pad2): track 0.00 -> 1.96 mm
- net GND: vias 0 -> 21
Other:
- board text added: "1.8V"
- board text added: "2.5V"
- board text added: "3.3V"
- board text added: "EXT"
- board text added: "Niklas Fauth Jan Henrik Hemsing 2019"
- board text added: "RST/RXD"
- board text added: "Tag-Connect Universal Adapter"
- board text removed: "SWD/UART"
- board text removed: "Tag- Connect"
- board text removed: "Universal Adapter"
